File: discipline-pcb.kicad_pcb (KiCad board)
At the start: 2 copper layers, 304.9 x 122.8 mm, 197 parts, among them J1 AVR-ISP-6, SW1 KEYSW, SW10 KEYSW, SW11 KEYSW, SW12 KEYSW, SW13 KEYSW, SW14 KEYSW, SW15 KEYSW, SW16 KEYSW, SW17 KEYSW, SW18 KEYSW, SW19 KEYSW, SW2 KEYSW, SW20 KEYSW, SW21 KEYSW, SW22 KEYSW, SW23 KEYSW, SW24 KEYSW, SW25 KEYSW, SW26 KEYSW, SW27 KEYSW, SW28 KEYSW, SW29 KEYSW, SW3 KEYSW, SW30 KEYSW, SW31 KEYSW, SW32 KEYSW, SW33 KEYSW, SW34 KEYSW, SW35 KEYSW, SW36 KEYSW, SW37 KEYSW, SW38 KEYSW, SW39 KEYSW, SW4 KEYSW, SW40 KEYSW, SW41 KEYSW, SW42 KEYSW, SW43 KEYSW, SW44 KEYSW, SW45 KEYSW, SW46 KEYSW, SW47 KEYSW, SW48 KEYSW, SW49 KEYSW, SW5 KEYSW, SW50 KEYSW, SW51 KEYSW, SW52 KEYSW, SW53 KEYSW, SW54 KEYSW, SW55 KEYSW, SW56 KEYSW, SW57 KEYSW, SW58 KEYSW, SW59 KEYSW, SW6 KEYSW, SW60 KEYSW, SW61 KEYSW, SW62 KEYSW, SW63 KEYSW, SW64 KEYSW, SW65 KEYSW, SW66 KEYSW, SW67 KEYSW, SW68 KEYSW, SW69 KEYSW, SW7 KEYSW, SW70 KEYSW, SW71 KEYSW, SW72 KEYSW, SW73 KEYSW, SW74 KEYSW, SW75 KEYSW, SW76 KEYSW, SW77 KEYSW, SW78 KEYSW, SW8 KEYSW, SW9 KEYSW, U1 ATmega32A-PU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

Commit message: Base design of Delight Keyboard
All traces are connected, it's not pretty, but it would work.
Parts:
- removed D71: , cftkb:D_DO-35_SOD27_P5.08mm_Horizontal
- removed the G*** at (354.1, 71.1)
- removed the G*** at (58.5, 71.1)
- removed the REF** at (57.8, 61.7)
- removed the REF** at (57.8, 80.4)
- removed the REF** at (206.2, 80.4)
- added D0: , cftkb:D_DO-35_SOD27_P5.08mm_Horizontal, F.Cu at (199.9, 68.1)
- added D75: , cftkb:D_DO-35_SOD27_P5.08mm_Horizontal, F.Cu at (217.7, 74.2)
- added REF**: MountingHole_2.2mm_M2_Pad, MountingHole:MountingHole_2.2mm_M2_Pad, F.Cu at (61.0, 123.4)
- added REF**: MountingHole_2.2mm_M2_Pad, MountingHole:MountingHole_2.2mm_M2_Pad, F.Cu at (76.5, 69.3)
- added SW0: KEYSW, cftkb:SW_Cherry_MX1A_1.00u_PCB-NOSCREEN, F.Cu at (65.9, 70.6)
- moved C4 240.4 mm to (85.9, 82.5), turned to 180 degrees
- moved C5 209.5 mm to (111.0, 77.7), turned to 180 degrees
- moved D59 207.2 mm to (74.7, 162.6), turned to 180 degrees
- moved C3 201.4 mm to (83.3, 79.5)
- moved U1 171.4 mm to (128.5, 83.1)
- moved R7 171.1 mm to (125.2, 83.1)
- moved USB1 170.0 mm to (107.7, 68.3)
- moved R1 169.9 mm to (120.1, 73.1)
- moved R2 169.9 mm to (120.1, 70.6)
- moved R3 169.9 mm to (125.2, 75.7)
- moved R4 169.9 mm to (125.2, 78.2)
- moved R5 169.9 mm to (125.2, 80.7)
- moved R6 169.9 mm to (120.1, 68.1)
- moved D61 169.6 mm to (116.1, 162.8), turned to 180 degrees
- moved D70 169.2 mm to (114.1, 76.7)
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Connections:
- D1 pad 1: row0 -> row1
- D16 pad 1: row1 -> row2
- D31 pad 1: row2 -> row3
- D45 pad 1: row3 -> row4
- SW59 pad 1: col0 -> col1
- SW60 pad 1: col1 -> col2
- SW61 pad 1: col2 -> col3
- SW70 pad 1: col0 -> col1
- SW71 pad 1: col2 -> col3
- U1 pad 1: row4 -> col5
- U1 pad 19: col5 -> row2
- U1 pad 2: row2 -> col6
- U1 pad 20: col6 -> row3
- U1 pad 21: col14 -> row1
- U1 pad 22: col13 -> row0
- U1 pad 23: col12 -> row4
- U1 pad 24: col11 -> col14
- U1 pad 25: col10 -> col13
- U1 pad 26: col9 -> col12
- U1 pad 27: col8 -> col11
- U1 pad 28: col7 -> col10
- U1 pad 3: row0 -> col7
- U1 pad 37: col2 -> col3
- U1 pad 38: col0 -> col2
- U1 pad 39: row1 -> col1
- U1 pad 4: col1 -> col8
- U1 pad 40: row3 -> col0
- U1 pad 5: col3 -> col9
Routing:
- net Net-(D59-Pad2): track 462.2 -> 9.92 mm
- net Net-(D61-Pad2): track 425.1 -> 22.3 mm
- net Net-(D62-Pad2): track 355.8 -> 15.4 mm
- net row4: track 299.4 -> 602.8 mm
- net Net-(D63-Pad2): track 279.4 -> 10.3 mm
- net Net-(D68-Pad2): track 232.5 -> 5.67 mm
- net Net-(D65-Pad2): track 215.1 -> 5.69 mm
- net col0: track 364.4 -> 161.2 mm, vias 2 -> 0
- net row3: track 404.8 -> 205.2 mm, vias 7 -> 0
- net GND: track 223.5 -> 28.8 mm, vias 48 -> 3
- net col2: track 331.4 -> 140.3 mm, vias 2 -> 1
- net Net-(D66-Pad2): track 190.5 -> 5.41 mm
- net Net-(D75-Pad2): track 15.0 -> 197.4 mm
- net Net-(D64-Pad2): track 188.7 -> 21.1 mm
- net col5: track 269.8 -> 102.9 mm
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Other:
- board size 304.9 x 122.8 mm -> 304.9 x 114.5 mm
- board text removed: "3.6V"
- board text removed: "500mA"
- board text removed: "ISP"
- board text removed: "ZENER DIODES"
