File: discipline-pcb.kicad_pcb (KiCad board)
At the start: 2 copper layers, 304.9 x 114.5 mm, 196 parts, among them J1 AVR-ISP-6, SW0 KEYSW, SW1 KEYSW, SW10 KEYSW, SW11 KEYSW, SW12 KEYSW, SW13 KEYSW, SW14 KEYSW, SW15 KEYSW, SW16 KEYSW, SW17 KEYSW, SW18 KEYSW, SW19 KEYSW, SW2 KEYSW, SW20 KEYSW, SW21 KEYSW, SW22 KEYSW, SW23 KEYSW, SW24 KEYSW, SW25 KEYSW, SW26 KEYSW, SW27 KEYSW, SW28 KEYSW, SW29 KEYSW, SW3 KEYSW, SW30 KEYSW, SW31 KEYSW, SW32 KEYSW, SW33 KEYSW, SW34 KEYSW, SW35 KEYSW, SW36 KEYSW, SW37 KEYSW, SW38 KEYSW, SW39 KEYSW, SW4 KEYSW, SW40 KEYSW, SW41 KEYSW, SW42 KEYSW, SW43 KEYSW, SW44 KEYSW, SW45 KEYSW, SW46 KEYSW, SW47 KEYSW, SW48 KEYSW, SW49 KEYSW, SW5 KEYSW, SW50 KEYSW, SW51 KEYSW, SW52 KEYSW, SW53 KEYSW, SW54 KEYSW, SW55 KEYSW, SW56 KEYSW, SW57 KEYSW, SW58 KEYSW, SW59 KEYSW, SW6 KEYSW, SW60 KEYSW, SW61 KEYSW, SW62 KEYSW, SW63 KEYSW, SW64 KEYSW, SW65 KEYSW, SW66 KEYSW, SW67 KEYSW, SW68 KEYSW, SW69 KEYSW, SW7 KEYSW, SW70 KEYSW, SW71 KEYSW, SW72 KEYSW, SW73 KEYSW, SW74 KEYSW, SW75 KEYSW, SW76 KEYSW, SW77 KEYSW, SW78 KEYSW, SW8 KEYSW, SW9 KEYSW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

Commit message: Front Side Cleanup
All major row/column wires are in a great spot now.
Parts:
- moved D16 0.25 mm to (205.0, 72.4)
- moved D17 0.25 mm to (212.6, 70.4)
- moved D18 0.25 mm to (222.8, 70.4)
- moved D19 0.25 mm to (232.7, 70.4)
- moved D20 0.25 mm to (242.6, 70.4)
- moved D32 0.25 mm to (215.1, 72.4)
- moved D33 0.25 mm to (225.3, 72.4)
- moved D34 0.25 mm to (235.2, 72.4)
- moved D35 0.25 mm to (245.1, 72.4)
- moved D0 0.25 mm to (199.9, 68.3)
- moved D1 0.25 mm to (202.4, 70.3)
- moved D2 0.25 mm to (210.1, 68.3)
- moved D3 0.25 mm to (220.2, 68.3)
- moved D31 0.25 mm to (207.5, 74.4)
- moved D4 0.25 mm to (230.1, 68.3)
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Routing:
- net Net-(D14-Pad2): track 23.1 -> 67.8 mm, vias 0 -> 1
- net Net-(D13-Pad2): track 60.0 -> 82.5 mm
- net Net-(D75-Pad2): track 197.4 -> 177.2 mm
- net Net-(D0-Pad2): track 149.8 -> 169.0 mm
- net Net-(D2-Pad2): track 142.1 -> 161.1 mm, vias 0 -> 1
- net Net-(D32-Pad2): track 174.0 -> 155.4 mm
- net Net-(D31-Pad2): track 186.6 -> 170.9 mm
- net Net-(D28-Pad2): track 44.9 -> 59.2 mm
- net Net-(D3-Pad2): track 139.7 -> 153.2 mm, vias 0 -> 1
- net Net-(D18-Pad2): track 144.1 -> 131.7 mm
- net Net-(D12-Pad2): track 71.2 -> 82.0 mm
- net Net-(D17-Pad2): track 154.5 -> 145.1 mm
- net Net-(D16-Pad2): track 162.6 -> 154.2 mm
- net Net-(D7-Pad2): track 123.8 -> 131.8 mm
- net Net-(D1-Pad2): track 149.5 -> 157.4 mm
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
Commit message: Last cleanup of placements.
Parts:
- added REF**: MountingHole_2.2mm_M2_Pad, MountingHole:MountingHole_2.2mm_M2_Pad, F.Cu at (76.5, 80.3)
- added REF**: MountingHole_2.2mm_M2_Pad, MountingHole:MountingHole_2.2mm_M2_Pad, F.Cu at (194.3, 81.8)
- moved REF** 12.4 mm to (194.1, 70.1)
- moved REF** 0.76 mm to (197.6, 109.2)
Connections:
- U1 pad 21: row1 -> row0
- U1 pad 22: row0 -> row1
Routing:
- net reset: track 83.3 -> 73.1 mm
- net row1: track 168.2 -> 172.3 mm
- net col10: track 212.7 -> 216.1 mm
- net Net-(D12-Pad2): track 82.0 -> 85.1 mm
- net Net-(D27-Pad2): track 58.8 -> 61.9 mm
- net row0: track 167.5 -> 164.4 mm
- net col4: track 105.7 -> 108.2 mm
- net col11: track 215.7 -> 218.0 mm
- net col3: track 138.5 -> 140.5 mm
- net col2: track 140.3 -> 141.8 mm
- net boot: track 89.9 -> 88.6 mm
- net col12: track 229.5 -> 230.7 mm
- net row3: track 204.3 -> 203.2 mm
- net row2: track 181.9 -> 181.1 mm
- net MISO: track 35.4 -> 35.9 mm
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
Commit message: More trace design
No more messing with it.
Parts:
- moved REF** 1.69 mm to (95.0, 160.5)
Routing:
- net Net-(D8-Pad2): track 130.5 -> 111.9 mm
- net Net-(D23-Pad2): track 107.0 -> 90.1 mm
- net Net-(D38-Pad2): track 115.6 -> 100.5 mm
- net row4: track 602.0 -> 591.8 mm
- net Net-(D18-Pad2): track 131.4 -> 140.3 mm
- net Net-(D7-Pad2): track 131.8 -> 125.3 mm
- net Net-(D27-Pad2): track 61.9 -> 55.8 mm
- net Net-(D12-Pad2): track 85.1 -> 79.2 mm
- net Net-(D22-Pad2): track 108.3 -> 103.6 mm
- net Net-(D51-Pad2): track 135.9 -> 131.9 mm
- net col10: track 216.1 -> 212.7 mm
- net Net-(D9-Pad2): track 110.3 -> 107.1 mm
- net col11: track 218.0 -> 214.9 mm
- net col12: track 230.7 -> 227.7 mm
- net Net-(D37-Pad2): track 117.0 -> 114.3 mm
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
Commit message: Wrapping Up
Finished up all major tasks.
Parts:
- removed the D12 at (310.2, 68.3)
- removed the D30 at (342.4, 70.4)
- removed the G*** at (155.1, 174.0) (x2)
- removed the G*** at (155.2, 174.0) (x2)
- removed the REF** at (76.5, 80.3)
- removed the REF** at (354.7, 80.4)
- removed the REF** at (354.7, 69.8)
- removed the REF** at (76.5, 69.3)
- removed the REF** at (194.3, 81.8)
- added D11: , cftkb:D_DO-35_SOD27_P5.08mm_Horizontal, F.Cu at (310.6, 68.3)
- added D29: , cftkb:D_DO-35_SOD27_P5.08mm_Horizontal, F.Cu at (343.7, 70.3)
- added REF**: MountingHole_2.2mm_M2_Pad, MountingHole:MountingHole_2.2mm_M2_Pad, F.Cu at (354.6, 81.8)
- added REF**: MountingHole_2.2mm_M2_Pad, MountingHole:MountingHole_2.2mm_M2_Pad, F.Cu at (354.6, 70.1)
- added REF**: MountingHole_2.2mm_M2_Pad, MountingHole:MountingHole_2.2mm_M2_Pad, F.Cu at (194.1, 81.8)
- added REF**: MountingHole_2.2mm_M2_Pad, MountingHole:MountingHole_2.2mm_M2_Pad, F.Cu at (76.5, 70.1)
- added REF**: MountingHole_2.2mm_M2_Pad, MountingHole:MountingHole_2.2mm_M2_Pad, F.Cu at (76.5, 81.8)
- G*** (x2): footprint logos:coseyfannitutti_16mm -> cftkb:lotier_rev1_16mm_mask
- G*** (x2): footprint logos:coseyfannitutti_rev1_16mm_copper -> cftkb:lotier_rev1_16mm_copper
- G*** (x2): footprint logos:DISCIPLINE_SMALL_COPPER -> cftkb:DELIGHT_SMALL_COPPER
- G*** (x2): footprint logos:DISCIPLINE_SMALL_MASK -> cftkb:DELIGHT_SMALL_MASK
- moved G*** 3.05 mm to (155.2, 166.7) (x4)
- moved G*** 2.55 mm to (155.5, 170.9) (x2)
- moved G*** 2.55 mm to (155.3, 170.9) (x2)
- moved D14 1.27 mm to (341.1, 68.3)
- moved D58 1.27 mm to (348.7, 74.4)
- moved D43 1.27 mm to (346.2, 72.4)
- moved REF** 1.14 mm to (197.1, 108.2)
- moved D2 1.02 mm to (219.2, 68.3)
- moved D17 1.02 mm to (221.7, 70.3)
- moved D16 1.02 mm to (211.6, 70.3)
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- renumbered D2 to D1, D11 to D10, D13 to D12, D14 to D13, D15 to D14, D1 to D15, D17 to D16, D18 to D17, D19 to D18, D20 to D19, D3 to D2, D21 to D20, D22 to D21, D23 to D22, D24 to D23, D25 to D24, D26 to D25, D27 to D26, D28 to D27, D29 to D28, D4 to D3, D16 to D30, D32 to D31, D33 to D32, D34 to D33, D35 to D34, D36 to D35, D37 to D36, D38 to D37, D39 to D38, D40 to D39, D5 to D4, D41 to D40, D42 to D41, D43 to D42, D44 to D43, D31 to D44, D75 to D45, D6 to D5, D45 to D59, D7 to D6, D59 to D60, D60 to D61, D61 to D62, D62 to D63, D63 to D64, D64 to D65, D68 to D66, D65 to D67, D66 to D68, D67 to D69, D8 to D7, D69 to D70, D70 to D71, D9 to D8, D10 to D9, SW61 to S62, SW2 to SW1, SW11 to SW10, SW12 to SW11, SW13 to SW12, SW14 to SW13, SW15 to SW14, SW1 to SW15, SW17 to SW16, SW18 to SW17, SW19 to SW18, SW20 to SW19, SW3 to SW2, SW21 to SW20, SW22 to SW21, SW23 to SW22, SW24 to SW23, SW25 to SW24, SW26 to SW25, SW27 to SW26, SW28 to SW27, SW29 to SW28, SW76 to SW28-2, SW30 to SW29, SW4 to SW3, SW16 to SW30, SW32 to SW31, SW33 to SW32, SW34 to SW33, SW35 to SW34, SW36 to SW35, SW37 to SW36, SW38 to SW37, SW39 to SW38, SW40 to SW39, SW5 to SW4, SW41 to SW40, SW42 to SW41, SW43 to SW42, SW77 to SW42-2, SW44 to SW43, SW31 to SW44, SW69 to SW44-2, SW75 to SW45, SW6 to SW5, SW45 to SW59, SW78 to SW59-2, SW7 to SW6, SW59 to SW60, SW70 to SW60-2, SW60 to SW61, SW71 to SW62-2, SW62 to SW63, SW72 to SW63-2, SW63 to SW64, SW73 to SW64-2, SW64 to SW65, SW74 to SW65-2, SW68 to SW66, SW65 to SW67, SW66 to SW68, SW67 to SW69, SW8 to SW7, SW9 to SW8, SW10 to SW9
Routing:
- net boot: track 88.6 -> 98.0 mm
- net row3: track 203.2 -> 209.3 mm
- net row4: track 591.8 -> 587.5 mm
- net row2: track 181.1 -> 183.2 mm
- net col4: track 108.2 -> 110.1 mm
- net col14: track 268.9 -> 270.7 mm
- net Net-(D11-Pad2): track 79.2 -> 77.7 mm
- net col3: track 140.5 -> 141.8 mm
- net Net-(D14-Pad2): track 20.5 -> 19.3 mm
- net row0: track 164.4 -> 165.5 mm
- net Net-(D1-Pad2): track 161.3 -> 160.3 mm
- net Net-(D30-Pad2): track 154.2 -> 153.1 mm
- net Net-(D44-Pad2): track 170.9 -> 169.9 mm
- net +5V: track 116.9 -> 117.9 mm
- net Net-(D58-Pad2): track 73.8 -> 73.1 mm
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Other:
- board text removed: "ISO"

Commit message: Cleanup of Files
Just removing a bunch of the files.
Other:
- rule pad_to_mask_clearance: 0.051 -> 0
