File: delight-pcb.kicad_pcb (KiCad board)
At the start: 2 copper layers, 304.9 x 114.5 mm, 194 parts, among them J1 AVR-ISP-6, SW0 KEYSW, SW1 KEYSW, SW10 KEYSW, SW11 KEYSW, SW12 KEYSW, SW13 KEYSW, SW14 KEYSW, SW15 KEYSW, SW16 KEYSW, SW17 KEYSW, SW18 KEYSW, SW19 KEYSW, SW2 KEYSW, SW20 KEYSW, SW21 KEYSW, SW22 KEYSW, SW23 KEYSW, SW24 KEYSW, SW25 KEYSW, SW26 KEYSW, SW27 KEYSW, SW28 KEYSW, SW28-2 KEYSW, SW29 KEYSW, SW3 KEYSW, SW30 KEYSW, SW31 KEYSW, SW32 KEYSW, SW33 KEYSW, SW34 KEYSW, SW35 KEYSW, SW36 KEYSW, SW37 KEYSW, SW38 KEYSW, SW39 KEYSW, SW4 KEYSW, SW40 KEYSW, SW41 KEYSW, SW42 KEYSW, SW42-2 KEYSW, SW43 KEYSW, SW44 KEYSW, SW44-2 KEYSW, SW45 KEYSW, SW46 KEYSW, SW47 KEYSW, SW48 KEYSW, SW49 KEYSW, SW5 KEYSW, SW50 KEYSW, SW51 KEYSW, SW52 KEYSW, SW53 KEYSW, SW54 KEYSW, SW55 KEYSW, SW56 KEYSW, SW57 KEYSW, SW58 KEYSW, SW59 KEYSW, SW59-2 KEYSW, SW6 KEYSW, SW60 KEYSW, SW60-2 KEYSW, SW61 KEYSW, SW62-2 KEYSW, SW63 KEYSW, SW63-2 KEYSW, SW64 KEYSW, SW64-2 KEYSW, SW65 KEYSW, SW65-2 KEYSW, SW66 KEYSW, SW67 KEYSW, SW68 KEYSW, SW69 KEYSW, SW7 KEYSW, SW8 KEYSW, SW9 KEYSW, U1 ATmega32A-PU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

Commit message: Attempted Project Rename
Attempting to rename the project.
Other:
- board text added: "DELIGHT - 65% keyboard assembled with only through hole components"
- board text removed: "DISCIPLINE - 65% keyboard assembled with only through hole components"
Changed lines of the file:
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@@
     (effects (font (size 1.5 1.5) (thickness 0.3)))
   )
-  (gr_text "DISCIPLINE - 65% keyboard assembled with only through hole components" (at 353.4156 261.2644) (layer Cmts.User)
+  (gr_text "DELIGHT - 65% keyboard assembled with only through hole components" (at 353.4156 261.2644) (layer Cmts.User)
     (effects (font (size 1.5 1.5) (thickness 0.3)))
   )
