File: board/delight-pcb.kicad_pcb (KiCad board)
At the start: 2 copper layers, 304.9 x 114.5 mm, 194 parts, among them J1 AVR-ISP-6, SW0 KEYSW, SW1 KEYSW, SW10 KEYSW, SW11 KEYSW, SW12 KEYSW, SW13 KEYSW, SW14 KEYSW, SW15 KEYSW, SW16 KEYSW, SW17 KEYSW, SW18 KEYSW, SW19 KEYSW, SW2 KEYSW, SW20 KEYSW, SW21 KEYSW, SW22 KEYSW, SW23 KEYSW, SW24 KEYSW, SW25 KEYSW, SW26 KEYSW, SW27 KEYSW, SW28 KEYSW, SW28-2 KEYSW, SW29 KEYSW, SW3 KEYSW, SW30 KEYSW, SW31 KEYSW, SW32 KEYSW, SW33 KEYSW, SW34 KEYSW, SW35 KEYSW, SW36 KEYSW, SW37 KEYSW, SW38 KEYSW, SW39 KEYSW, SW4 KEYSW, SW40 KEYSW, SW41 KEYSW, SW42 KEYSW, SW42-2 KEYSW, SW43 KEYSW, SW44 KEYSW, SW44-2 KEYSW, SW45 KEYSW, SW46 KEYSW, SW47 KEYSW, SW48 KEYSW, SW49 KEYSW, SW5 KEYSW, SW50 KEYSW, SW51 KEYSW, SW52 KEYSW, SW53 KEYSW, SW54 KEYSW, SW55 KEYSW, SW56 KEYSW, SW57 KEYSW, SW58 KEYSW, SW59 KEYSW, SW59-2 KEYSW, SW6 KEYSW, SW60 KEYSW, SW60-2 KEYSW, SW61 KEYSW, SW62-2 KEYSW, SW63 KEYSW, SW63-2 KEYSW, SW64 KEYSW, SW64-2 KEYSW, SW65 KEYSW, SW65-2 KEYSW, SW66 KEYSW, SW67 KEYSW, SW68 KEYSW, SW69 KEYSW, SW7 KEYSW, SW8 KEYSW, SW9 KEYSW, U1 ATmega32A-PU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

Commit message: Start Process to design hotswap
Parts:
- moved U1 5.08 mm to (133.6, 83.1)
- moved D71 4.79 mm to (118.9, 76.0)
- moved R6 3.90 mm to (122.9, 70.8)
- moved R2 3.64 mm to (122.9, 68.3)
- moved C3 2.93 mm to (86.1, 78.7), turned to 180 degrees
- moved R1 2.80 mm to (122.9, 73.2)
- moved R5 2.80 mm to (128.0, 80.6)
- moved R4 2.79 mm to (128.0, 78.1)
- moved R3 2.79 mm to (128.0, 75.7)
- moved R7 2.79 mm to (128.0, 83.1)
- moved LED1 2.70 mm to (119.4, 70.6)
- moved USB 2.62 mm to (109.0, 66.0)
- moved D63 2.34 mm to (186.9, 160.3)
- moved C4 2.30 mm to (88.1, 82.8)
- moved BOOT1 1.52 mm to (94.5, 68.3)
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- renumbered USB1 to USB
Routing:
- net GND: track 28.8 -> 8.36 mm, vias 23 -> 22
- net col1: track 184.4 -> 164.2 mm, vias 1 -> 0
- net SCK: track 58.8 -> 43.7 mm
- net reset: track 73.1 -> 83.3 mm, vias 0 -> 2
- net col4: track 110.1 -> 100.0 mm, vias 1 -> 0
- net col0: track 160.3 -> 165.9 mm
- net row4: track 587.5 -> 582.2 mm
- net Net-(C2-Pad1): track 41.7 -> 36.5 mm
- net row2: track 183.2 -> 178.1 mm
- net row3: track 209.3 -> 204.2 mm
- net row1: track 172.9 -> 167.9 mm
- net row0: track 165.5 -> 160.4 mm
- net col9: track 198.2 -> 193.1 mm
- net col7: track 135.4 -> 130.3 mm
- net Net-(C1-Pad1): track 39.6 -> 34.6 mm
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Other:
- board text removed: "POWER"

Commit message: Startup For Using standard library
Parts:
- BOOT1, RESET1: footprint cftkb:SW_PUSH_6mm -> Button_Switch_THT:SW_PUSH_6mm
- D0, D1, D10, D11, D12, D13, D14, D15, D16, D17, D18, D19, D2, D20, D21, D22, D23, D24, D25, D26, D27, D28, D29, D3, D30, D31, D32, D33, D34, D35, D36, D37, D38, D39, D4, D40, D41, D42, D43, D44, D45, D46, D47, D48, D49, D5, D50, D51, D52, D53, D54, D55, D56, D57, D58, D59, D6, D60, D61, D62, D63, D64, D65, D66, D67, D68, D69, D7, D70, D71, D8, D9: footprint cftkb:D_DO-35_SOD27_P5.08mm_Horizontal -> Diode_THT:D_DO-35_SOD27_P7.62mm_Horizontal
- J1: footprint cftkb:AVR_ICSP_3x2 -> Connector_PinHeader_2.54mm:PinHeader_2x03_P2.54mm_Vertical
- LED1: footprint cftkb:LED_D3.0mm -> LED_THT:LED_D3.0mm
- U1: footprint cftkb:DIP-40_W15.24mm -> Package_DIP:DIP-40_W15.24mm
- USB: value USB_C_GCT_USB4085 -> USB_C_Receptacle_GCT_USB4085; footprint cftkb:USB_C_GCT_USB4085 -> Connector_USB:USB_C_Receptacle_GCT_USB4085
- moved USB 6.79 mm to (111.9, 72.2)
- moved J1 2.62 mm to (112.0, 80.5), turned to 270 degrees
Routing:
- net +5V: track 118.5 -> 116.8 mm
- net col1: track 164.2 -> 163.1 mm
- net Net-(D71-Pad1): track 28.9 -> 29.5 mm
- net boot: track 100.6 -> 101.1 mm
- net reset: vias 2 -> 1
- net GND: vias 22 -> 23

Commit message: Swapped out as many custom mods for standard.
Parts:
- removed D59, D60, D61, D62, D63, D64, D65, D66, D67, D68, D69: , Diode_THT:D_DO-35_SOD27_P7.62mm_Horizontal
- removed G*** (x2): LOGO, cftkb:lotier_rev1_16mm_mask
- removed G*** (x2): LOGO, cftkb:lotier_rev1_16mm_copper
- removed G*** (x2): LOGO, cftkb:DELIGHT_SMALL_COPPER
- removed G*** (x2): LOGO, cftkb:DELIGHT_SMALL_MASK
- removed the REF** at (197.1, 108.2)
- removed the REF** at (298.7, 104.3)
- removed the REF** at (107.7, 104.1)
- removed the REF** at (316.2, 161.1)
- removed the REF** at (95.0, 160.8)
- removed the REF** at (61.0, 123.4)
- removed the REF** at (184.8, 171.0)
- removed the REF** at (206.2, 167.0)
- removed S62, SW44-2, SW59-2, SW60, SW61, SW64, SW65: KEYSW, cftkb:SW_Cherry_MX1A_1.25u_PCBNOSCREEN
- removed ST72: 7U, cftkb:MX-7U-Stabilizer
- removed SW0, SW1, SW10, SW11, SW12, SW14, SW15, SW16, SW17, SW18, SW19, SW2, SW20, SW21, SW22, SW23, SW24, SW25, SW26, SW27, SW29, SW3, SW31, SW32, SW33, SW34, SW35, SW36, SW37, SW38, SW39, SW4, SW40, SW41, SW42-2, SW43, SW45, SW46, SW47, SW48, SW49, SW5, SW50, SW51, SW52, SW53, SW54, SW55, SW57, SW58, SW6, SW63, SW63-2, SW66, SW67, SW68, SW69, SW7, SW8, SW9: KEYSW, cftkb:SW_Cherry_MX1A_1.00u_PCB-NOSCREEN
- removed SW13: KEYSW, cftkb:SW_Cherry_MX1A_2.00u_PCBNOSCREEN
- removed SW28, SW30, SW60-2, SW62-2, SW64-2, SW65-2: KEYSW, cftkb:SW_Cherry_MX1A_1.50u_PCBNOSCREEN
- removed SW28-2: KEYSW, cftkb:SW_Cherry_MX1A_ISOEnter_PCB_ReversedStabilizer
- removed SW42, SW59: KEYSW, cftkb:SW_Cherry_MX1A_2.25u_PCBNOSCREEN
- removed SW44, SW56: KEYSW, cftkb:SW_Cherry_MX1A_1.75u_PCBNOSCREEN
- C1, C2: footprint cftkb:C_Disc_D3.0mm_W1.6mm_P2.50mm -> Capacitor_THT:C_Disc_D3.0mm_W1.6mm_P2.50mm
- C3: footprint cftkb:CP_Radial_D4.0mm_P1.50mm -> Capacitor_THT:CP_Radial_D4.0mm_P1.50mm
- C4, C5: footprint cftkb:C_Disc_D4.3mm_W1.9mm_P5.00mm -> Capacitor_THT:C_Disc_D4.3mm_W1.9mm_P5.00mm
- F1: footprint cftkb:polyfuse_5.1mm -> project:Bourns-MF-R050-0-0-MFG
- R1, R2, R3, R4, R5, R6, R7: footprint cftkb:R_Axial_DIN0204_L3.6mm_D1.6mm_P5.08mm_Horizontal -> Resistor_THT:R_Axial_DIN0204_L3.6mm_D1.6mm_P5.08mm_Horizontal
- Y1: footprint cftkb:Crystal_HC49-4H_Vertical -> Crystal:Crystal_HC49-4H_Vertical
- moved R1 5.12 mm to (128.0, 73.2), turned to 180 degrees
Routing:
- net row4: track 582.2 -> 263.0 mm
- net col14: track 266.5 -> 22.0 mm
- net col13: track 264.0 -> 23.5 mm
- net col12: track 225.0 -> 24.9 mm
- net col9: track 193.1 -> 4.82 mm
- net col11: track 211.5 -> 26.3 mm
- net col10: track 208.5 -> 27.7 mm
- net Net-(D45-Pad2): track 176.4 -> 2.80 mm
- net Net-(D46-Pad2): track 172.3 -> 11.0 mm
- net Net-(D47-Pad2): track 162.0 -> 3.35 mm
- net Net-(D44-Pad2): track 169.9 -> 14.7 mm
- net Net-(D0-Pad2): track 167.5 -> 13.7 mm
- net Net-(D31-Pad2): track 154.7 -> 7.09 mm
- net Net-(D48-Pad2): track 154.3 -> 8.38 mm
- net Net-(D15-Pad2): track 155.9 -> 13.1 mm
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Other:
- board size 304.9 x 114.5 mm -> 301.6 x 111.2 mm
- board text removed: "1.25U"
- board text removed: "1.25U ISO"
- board text removed: "1.5U"
- board text removed: "1U"
- board text removed: "1U ISO"
- board text removed: "2.25U ANSI"
- board text removed: "ANSI ENTER"
- board text removed: "ISO ENTER"
- board text removed: "STANDARD"
- board text removed: "STEPPED"

Commit message: Cleaning up layout.
Routing:
- net row3: track 204.2 -> 0.00 mm
- net row2: track 178.1 -> 0.00 mm
- net row1: track 167.9 -> 25.0 mm
- net row0: track 160.4 -> 17.6 mm
- net Net-(D57-Pad2): track 56.3 -> 0.00 mm
- net Net-(D42-Pad2): track 42.6 -> 0.00 mm
- net Net-(D2-Pad2): track 31.0 -> 0.00 mm
- net Net-(D13-Pad2): track 30.1 -> 0.00 mm
- net Net-(D28-Pad2): track 27.4 -> 0.00 mm
- net Net-(D1-Pad2): track 22.9 -> 0.00 mm
- net Net-(D12-Pad2): track 22.9 -> 0.00 mm
- net Net-(D4-Pad2): track 21.2 -> 0.00 mm
- net Net-(D8-Pad2): track 20.3 -> 0.00 mm
- net Net-(D27-Pad2): track 20.2 -> 0.00 mm
- net Net-(D6-Pad2): track 19.6 -> 0.00 mm
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
Commit message: Update delight-pcb.kicad_pcb
Parts:
- added D59: , cftkb:D_DO-35_SOD27_P5.08mm_Horizontal, F.Cu at (85.6, 154.9)
- added D60: , cftkb:D_DO-35_SOD27_P5.08mm_Horizontal, F.Cu at (85.6, 174.0)
- added D61: , cftkb:D_DO-35_SOD27_P5.08mm_Horizontal, F.Cu at (117.6, 174.2)
- added D62: , cftkb:D_DO-35_SOD27_P5.08mm_Horizontal, F.Cu at (127.0, 174.2)
- added D63: , cftkb:D_DO-35_SOD27_P5.08mm_Horizontal, F.Cu at (197.4, 174.0)
- added D64: , cftkb:D_DO-35_SOD27_P5.08mm_Horizontal, F.Cu at (271.8, 174.5)
- added D65: , cftkb:D_DO-35_SOD27_P5.08mm_Horizontal, F.Cu at (286.5, 174.2)
- added D66: , cftkb:D_DO-35_SOD27_P5.08mm_Horizontal, F.Cu at (305.3, 174.2)
- added D67: , cftkb:D_DO-35_SOD27_P5.08mm_Horizontal, F.Cu at (324.6, 174.2)
- added D68: , cftkb:D_DO-35_SOD27_P5.08mm_Horizontal, F.Cu at (343.4, 174.5)
- added D69: , cftkb:D_DO-35_SOD27_P5.08mm_Horizontal, F.Cu at (362.5, 174.5)
- added G***: LOGO, cftkb:lotier_rev1_16mm_mask, B.Cu at (166.5, 182.3)
- added G***: LOGO, cftkb:lotier_rev1_16mm_mask, F.Cu at (166.3, 182.3)
- added G***: LOGO, cftkb:lotier_rev1_16mm_copper, B.Cu at (166.5, 182.3)
- added G***: LOGO, cftkb:lotier_rev1_16mm_copper, F.Cu at (166.3, 182.3)
- added G***: LOGO, cftkb:DELIGHT_SMALL_COPPER, F.Cu at (166.1, 178.1)
- added G***: LOGO, cftkb:DELIGHT_SMALL_COPPER, B.Cu at (166.1, 178.1)
- added G***: LOGO, cftkb:DELIGHT_SMALL_MASK, F.Cu at (166.1, 178.1)
- added G***: LOGO, cftkb:DELIGHT_SMALL_MASK, B.Cu at (166.1, 178.1)
- added REF**: MountingHole_2.2mm_M2_Pad, MountingHole:MountingHole_2.2mm_M2_Pad, F.Cu at (208.0, 119.6)
- added REF**: MountingHole_2.2mm_M2_Pad, MountingHole:MountingHole_2.2mm_M2_Pad, F.Cu at (309.6, 115.7)
- added REF**: MountingHole_2.2mm_M2_Pad, MountingHole:MountingHole_2.2mm_M2_Pad, F.Cu at (118.6, 115.6)
- added REF**: MountingHole_2.2mm_M2_Pad, MountingHole:MountingHole_2.2mm_M2_Pad, F.Cu at (327.2, 172.6)
- added REF**: MountingHole_2.2mm_M2_Pad, MountingHole:MountingHole_2.2mm_M2_Pad, F.Cu at (105.9, 172.2)
- added REF**: MountingHole_2.2mm_M2_Pad, MountingHole:MountingHole_2.2mm_M2_Pad, F.Cu at (71.9, 134.9)
- added REF**: 6.25U, cftkb:MX-6.25U-Stabilizer, F.Cu at (195.7, 182.4)
- added REF**: MountingHole_2.2mm_M2_Pad, MountingHole:MountingHole_2.2mm_M2_Pad, F.Cu at (217.1, 178.4)
- added S62: KEYSW, cftkb:SW_Cherry_MX1A_1.25u_PCBNOSCREEN, F.Cu at (126.8, 177.3)
- added ST72: 7U, cftkb:MX-7U-Stabilizer, F.Cu at (188.6, 182.4)
- added SW0: KEYSW, cftkb:SW_Cherry_MX1A_1.00u_PCB-NOSCREEN, F.Cu at (76.8, 82.0)
- added SW1: KEYSW, cftkb:SW_Cherry_MX1A_1.00u_PCB-NOSCREEN, F.Cu at (95.9, 101.1)
- added SW10: KEYSW, cftkb:SW_Cherry_MX1A_1.00u_PCB-NOSCREEN, F.Cu at (267.3, 101.1)
- added SW11: KEYSW, cftkb:SW_Cherry_MX1A_1.00u_PCB-NOSCREEN, F.Cu at (286.4, 101.1)
- added SW12: KEYSW, cftkb:SW_Cherry_MX1A_1.00u_PCB-NOSCREEN, F.Cu at (305.4, 101.1)
- added SW13: KEYSW, cftkb:SW_Cherry_MX1A_2.00u_PCBNOSCREEN, F.Cu at (334.0, 101.1)
- added SW14: KEYSW, cftkb:SW_Cherry_MX1A_1.00u_PCB-NOSCREEN, F.Cu at (362.6, 101.1)
- added SW15: KEYSW, cftkb:SW_Cherry_MX1A_1.00u_PCB-NOSCREEN, F.Cu at (76.8, 101.1)
- added SW16: KEYSW, cftkb:SW_Cherry_MX1A_1.00u_PCB-NOSCREEN, F.Cu at (105.4, 120.2)
- added SW17: KEYSW, cftkb:SW_Cherry_MX1A_1.00u_PCB-NOSCREEN, F.Cu at (124.4, 120.2)
- added SW18: KEYSW, cftkb:SW_Cherry_MX1A_1.00u_PCB-NOSCREEN, F.Cu at (143.5, 120.2)
- added SW19: KEYSW, cftkb:SW_Cherry_MX1A_1.00u_PCB-NOSCREEN, F.Cu at (162.5, 120.2)
- added SW2: KEYSW, cftkb:SW_Cherry_MX1A_1.00u_PCB-NOSCREEN, F.Cu at (114.9, 101.1)
- added SW20: KEYSW, cftkb:SW_Cherry_MX1A_1.00u_PCB-NOSCREEN, F.Cu at (181.6, 120.2)
- added SW21: KEYSW, cftkb:SW_Cherry_MX1A_1.00u_PCB-NOSCREEN, F.Cu at (200.6, 120.2)
- added SW22: KEYSW, cftkb:SW_Cherry_MX1A_1.00u_PCB-NOSCREEN, F.Cu at (219.7, 120.2)
- added SW23: KEYSW, cftkb:SW_Cherry_MX1A_1.00u_PCB-NOSCREEN, F.Cu at (238.7, 120.2)
- added SW24: KEYSW, cftkb:SW_Cherry_MX1A_1.00u_PCB-NOSCREEN, F.Cu at (257.8, 120.2)
- added SW25: KEYSW, cftkb:SW_Cherry_MX1A_1.00u_PCB-NOSCREEN, F.Cu at (276.8, 120.2)
- added SW26: KEYSW, cftkb:SW_Cherry_MX1A_1.00u_PCB-NOSCREEN, F.Cu at (295.9, 120.2)
- added SW27: KEYSW, cftkb:SW_Cherry_MX1A_1.00u_PCB-NOSCREEN, F.Cu at (314.9, 120.2)
- added SW28: KEYSW, cftkb:SW_Cherry_MX1A_1.50u_PCBNOSCREEN, F.Cu at (338.7, 120.2)
- added SW28-2: KEYSW, cftkb:SW_Cherry_MX1A_ISOEnter_PCB_ReversedStabilizer, F.Cu at (341.1, 129.7)
- added SW29: KEYSW, cftkb:SW_Cherry_MX1A_1.00u_PCB-NOSCREEN, F.Cu at (362.6, 120.2)
- added SW3: KEYSW, cftkb:SW_Cherry_MX1A_1.00u_PCB-NOSCREEN, F.Cu at (134.0, 101.1)
- added SW30: KEYSW, cftkb:SW_Cherry_MX1A_1.50u_PCBNOSCREEN, F.Cu at (81.6, 120.2)
- added SW31: KEYSW, cftkb:SW_Cherry_MX1A_1.00u_PCB-NOSCREEN, F.Cu at (110.1, 139.2)
- added SW32: KEYSW, cftkb:SW_Cherry_MX1A_1.00u_PCB-NOSCREEN, F.Cu at (129.2, 139.2)
- added SW33: KEYSW, cftkb:SW_Cherry_MX1A_1.00u_PCB-NOSCREEN, F.Cu at (148.2, 139.2)
- added SW34: KEYSW, cftkb:SW_Cherry_MX1A_1.00u_PCB-NOSCREEN, F.Cu at (167.3, 139.2)
- added SW35: KEYSW, cftkb:SW_Cherry_MX1A_1.00u_PCB-NOSCREEN, F.Cu at (186.3, 139.2)
- added SW36: KEYSW, cftkb:SW_Cherry_MX1A_1.00u_PCB-NOSCREEN, F.Cu at (205.4, 139.2)
- added SW37: KEYSW, cftkb:SW_Cherry_MX1A_1.00u_PCB-NOSCREEN, F.Cu at (224.4, 139.2)
- added SW38: KEYSW, cftkb:SW_Cherry_MX1A_1.00u_PCB-NOSCREEN, F.Cu at (243.5, 139.2)
- added SW39: KEYSW, cftkb:SW_Cherry_MX1A_1.00u_PCB-NOSCREEN, F.Cu at (262.5, 139.2)
- added SW4: KEYSW, cftkb:SW_Cherry_MX1A_1.00u_PCB-NOSCREEN, F.Cu at (153.0, 101.1)
- added SW40: KEYSW, cftkb:SW_Cherry_MX1A_1.00u_PCB-NOSCREEN, F.Cu at (281.6, 139.2)
- added SW41: KEYSW, cftkb:SW_Cherry_MX1A_1.00u_PCB-NOSCREEN, F.Cu at (300.6, 139.2)
- added SW42: KEYSW, cftkb:SW_Cherry_MX1A_2.25u_PCBNOSCREEN, F.Cu at (331.6, 139.2)
- added SW42-2: KEYSW, cftkb:SW_Cherry_MX1A_1.00u_PCB-NOSCREEN, F.Cu at (319.7, 139.2)
- added SW43: KEYSW, cftkb:SW_Cherry_MX1A_1.00u_PCB-NOSCREEN, F.Cu at (362.6, 139.2)
- added SW44: KEYSW, cftkb:SW_Cherry_MX1A_1.75u_PCBNOSCREEN, F.Cu at (83.9, 139.2)
- added SW44-2: KEYSW, cftkb:SW_Cherry_MX1A_1.25u_PCBNOSCREEN, F.Cu at (79.2, 139.2)
- added SW45: KEYSW, cftkb:SW_Cherry_MX1A_1.00u_PCB-NOSCREEN, F.Cu at (100.6, 158.3)
- added SW46: KEYSW, cftkb:SW_Cherry_MX1A_1.00u_PCB-NOSCREEN, F.Cu at (119.7, 158.3)
- added SW47: KEYSW, cftkb:SW_Cherry_MX1A_1.00u_PCB-NOSCREEN, F.Cu at (138.7, 158.3)
- added SW48: KEYSW, cftkb:SW_Cherry_MX1A_1.00u_PCB-NOSCREEN, F.Cu at (157.8, 158.3)
- added SW49: KEYSW, cftkb:SW_Cherry_MX1A_1.00u_PCB-NOSCREEN, F.Cu at (176.8, 158.3)
- added SW5: KEYSW, cftkb:SW_Cherry_MX1A_1.00u_PCB-NOSCREEN, F.Cu at (172.1, 101.1)
- added SW50: KEYSW, cftkb:SW_Cherry_MX1A_1.00u_PCB-NOSCREEN, F.Cu at (195.9, 158.3)
- added SW51: KEYSW, cftkb:SW_Cherry_MX1A_1.00u_PCB-NOSCREEN, F.Cu at (214.9, 158.3)
- added SW52: KEYSW, cftkb:SW_Cherry_MX1A_1.00u_PCB-NOSCREEN, F.Cu at (234.0, 158.3)
- added SW53: KEYSW, cftkb:SW_Cherry_MX1A_1.00u_PCB-NOSCREEN, F.Cu at (253.0, 158.3)
- added SW54: KEYSW, cftkb:SW_Cherry_MX1A_1.00u_PCB-NOSCREEN, F.Cu at (272.1, 158.3)
- added SW55: KEYSW, cftkb:SW_Cherry_MX1A_1.00u_PCB-NOSCREEN, F.Cu at (291.1, 158.3)
- added SW56: KEYSW, cftkb:SW_Cherry_MX1A_1.75u_PCBNOSCREEN, F.Cu at (317.3, 158.3)
- added SW57: KEYSW, cftkb:SW_Cherry_MX1A_1.00u_PCB-NOSCREEN, F.Cu at (343.5, 158.3)
- added SW58: KEYSW, cftkb:SW_Cherry_MX1A_1.00u_PCB-NOSCREEN, F.Cu at (362.6, 158.3)
- added SW59: KEYSW, cftkb:SW_Cherry_MX1A_2.25u_PCBNOSCREEN, F.Cu at (88.7, 158.3)
- added SW59-2: KEYSW, cftkb:SW_Cherry_MX1A_1.25u_PCBNOSCREEN, F.Cu at (79.2, 158.3)
- added SW6: KEYSW, cftkb:SW_Cherry_MX1A_1.00u_PCB-NOSCREEN, F.Cu at (191.1, 101.1)
- added SW60: KEYSW, cftkb:SW_Cherry_MX1A_1.25u_PCBNOSCREEN, F.Cu at (79.2, 177.3)
- added SW60-2: KEYSW, cftkb:SW_Cherry_MX1A_1.50u_PCBNOSCREEN, F.Cu at (81.6, 177.3)
- added SW61: KEYSW, cftkb:SW_Cherry_MX1A_1.25u_PCBNOSCREEN, F.Cu at (103.0, 177.3)
- added SW62-2: KEYSW, cftkb:SW_Cherry_MX1A_1.50u_PCBNOSCREEN, F.Cu at (110.2, 177.3)
- added SW63: KEYSW, cftkb:SW_Cherry_MX1A_1.00u_PCB-NOSCREEN, F.Cu at (198.2, 177.3)
- added SW63-2: KEYSW, cftkb:SW_Cherry_MX1A_1.00u_PCB-NOSCREEN, F.Cu at (191.1, 177.3)
- added SW64: KEYSW, cftkb:SW_Cherry_MX1A_1.25u_PCBNOSCREEN, F.Cu at (267.3, 177.3)
- added SW64-2: KEYSW, cftkb:SW_Cherry_MX1A_1.50u_PCBNOSCREEN, F.Cu at (272.1, 177.3)
- added SW65: KEYSW, cftkb:SW_Cherry_MX1A_1.25u_PCBNOSCREEN, F.Cu at (286.4, 177.3)
- added SW65-2: KEYSW, cftkb:SW_Cherry_MX1A_1.50u_PCBNOSCREEN, F.Cu at (300.7, 177.3)
- added SW66: KEYSW, cftkb:SW_Cherry_MX1A_1.00u_PCB-NOSCREEN, F.Cu at (305.4, 177.3)
- added SW67: KEYSW, cftkb:SW_Cherry_MX1A_1.00u_PCB-NOSCREEN, F.Cu at (324.5, 177.3)
- added SW68: KEYSW, cftkb:SW_Cherry_MX1A_1.00u_PCB-NOSCREEN, F.Cu at (343.5, 177.3)
- added SW69: KEYSW, cftkb:SW_Cherry_MX1A_1.00u_PCB-NOSCREEN, F.Cu at (362.6, 177.3)
- added SW7: KEYSW, cftkb:SW_Cherry_MX1A_1.00u_PCB-NOSCREEN, F.Cu at (210.2, 101.1)
- added SW8: KEYSW, cftkb:SW_Cherry_MX1A_1.00u_PCB-NOSCREEN, F.Cu at (229.2, 101.1)
- added SW9: KEYSW, cftkb:SW_Cherry_MX1A_1.00u_PCB-NOSCREEN, F.Cu at (248.3, 101.1)
- moved D11 15.8 mm to (321.6, 79.8)
- moved D13 15.8 mm to (341.9, 79.8)
- moved D18 15.8 mm to (242.8, 81.8)
- moved D22 15.8 mm to (283.5, 81.8)
- moved D23 15.8 mm to (293.6, 81.8)
- moved D25 15.8 mm to (313.9, 81.8)
- moved D27 15.8 mm to (334.3, 81.8)
- moved D29 15.8 mm to (354.6, 81.8)
- moved D48 15.8 mm to (258.1, 85.9)
- moved D50 15.8 mm to (278.4, 85.9)
- moved D52 15.8 mm to (298.7, 85.9)
- moved D54 15.8 mm to (319.0, 85.9)
- moved D55 15.8 mm to (329.2, 85.9)
- moved D57 15.8 mm to (349.5, 85.9)
- moved D6 15.8 mm to (270.8, 79.8)
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Routing:
- net row4: track 263.0 -> 600.2 mm
- net col14: track 22.0 -> 266.4 mm
- net col13: track 23.5 -> 263.9 mm
- net col12: track 24.9 -> 225.4 mm
- net col9: track 4.82 -> 193.0 mm
- net col11: track 26.3 -> 211.9 mm
- net col10: track 27.7 -> 208.7 mm
- net row2: track 0.00 -> 179.0 mm
- net row3: track 0.00 -> 176.9 mm
- net Net-(D45-Pad2): track 0.00 -> 175.1 mm
- net Net-(D46-Pad2): track 0.00 -> 171.1 mm
- net Net-(D44-Pad2): track 0.00 -> 169.4 mm
- net Net-(D0-Pad2): track 0.00 -> 166.4 mm
- net Net-(D47-Pad2): track 0.00 -> 160.8 mm
- net Net-(D1-Pad2): track 0.00 -> 159.5 mm, vias 0 -> 1
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Other:
- board size 301.6 x 111.2 mm -> 304.9 x 114.5 mm
- board text added: "1.25U"
- board text added: "1.25U ISO"
- board text added: "1.5U"
- board text added: "1U"
- board text added: "1U ISO"
- board text added: "2.25U ANSI"
- board text added: "ANSI ENTER"
- board text added: "ISO ENTER"
- board text added: "STANDARD"
- board text added: "STEPPED"

Commit message: Updated all routes.
Parts:
- USB1: renamed from USB; value USB_C_Receptacle_GCT_USB4085 -> USB_C_GCT_USB4085
Connections:
- U1 pad 19: row2 -> row3
- U1 pad 20: row3 -> row2
Routing:
- net row2: track 179.0 -> 174.5 mm
- net Net-(D4-Pad2): track 144.0 -> 140.2 mm
- net row3: track 176.9 -> 178.6 mm
- net col10: track 208.7 -> 210.2 mm
- net Net-(D53-Pad2): track 105.4 -> 104.1 mm
- net col11: track 211.9 -> 213.2 mm
- net Net-(D52-Pad2): track 117.6 -> 116.2 mm
- net Net-(D38-Pad2): track 95.6 -> 94.3 mm
- net Net-(D56-Pad2): track 80.4 -> 79.2 mm
- net col12: track 225.4 -> 226.6 mm
- net D+: track 45.8 -> 46.9 mm
- net col13: track 263.9 -> 264.9 mm
- net col14: track 266.4 -> 267.3 mm
- net Net-(D0-Pad2): track 166.4 -> 167.3 mm
- net Net-(D15-Pad2): track 154.9 -> 155.7 mm
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
Commit message: More cleanup
Parts:
- S62, SW44-2, SW59-2, SW60, SW61, SW64, SW65: footprint cftkb:SW_Cherry_MX1A_1.25u_PCBNOSCREEN -> cherrymx:SW_Cherry_MX_PCB_1.25u
- SW0, SW1, SW10, SW11, SW12, SW14, SW15, SW16, SW17, SW18, SW19, SW2, SW20, SW21, SW22, SW23, SW24, SW25, SW26, SW27, SW29, SW3, SW31, SW32, SW33, SW34, SW35, SW36, SW37, SW38, SW39, SW4, SW40, SW41, SW42-2, SW43, SW45, SW46, SW47, SW48, SW49, SW5, SW50, SW51, SW52, SW53, SW54, SW55, SW57, SW58, SW6, SW63, SW63-2, SW66, SW67, SW68, SW69, SW7, SW8, SW9: footprint cftkb:SW_Cherry_MX1A_1.00u_PCB-NOSCREEN -> cherrymx:SW_Cherry_MX_PCB_1.00u
- SW13: footprint cftkb:SW_Cherry_MX1A_2.00u_PCBNOSCREEN -> cherrymx:SW_Cherry_MX_PCB_2.00u
- SW28, SW30, SW60-2, SW62-2, SW64-2, SW65-2: footprint cftkb:SW_Cherry_MX1A_1.50u_PCBNOSCREEN -> cherrymx:SW_Cherry_MX_PCB_1.50u
- SW28-2: footprint cftkb:SW_Cherry_MX1A_ISOEnter_PCB_ReversedStabilizer -> cherrymx:SW_Cherry_MX_Plate_ISOEnter
- SW42, SW59: footprint cftkb:SW_Cherry_MX1A_2.25u_PCBNOSCREEN -> cherrymx:SW_Cherry_MX_PCB_2.25u
- SW44, SW56: footprint cftkb:SW_Cherry_MX1A_1.75u_PCBNOSCREEN -> cherrymx:SW_Cherry_MX_PCB_1.75u
- moved SW64 5.72 mm to (264.8, 182.4)
- moved SW64-2 5.71 mm to (269.6, 182.4)
- moved SW13 5.71 mm to (331.4, 106.2)
- moved SW28 5.69 mm to (336.2, 125.3)
- moved SW28-2 5.69 mm to (338.6, 134.8)
- moved SW42 5.68 mm to (329.1, 144.3)
- moved SW36 5.68 mm to (202.9, 144.3)
- moved SW39 5.68 mm to (260.0, 144.3)
- moved SW40 5.68 mm to (279.1, 144.3)
- moved SW63 5.68 mm to (195.7, 182.4)
- moved SW66 5.68 mm to (302.9, 182.4)
- moved SW67 5.68 mm to (321.9, 182.4)
- moved SW32 5.68 mm to (126.7, 144.3)
- moved SW11 5.68 mm to (283.8, 106.2)
- moved SW12 5.68 mm to (302.9, 106.2)
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Connections:
- S62 pad 1: col3 -> Net-(D62-Pad2)
- S62 pad 2: Net-(D62-Pad2) -> col3
- SW0 pad 1: col0 -> Net-(D0-Pad2)
- SW0 pad 2: Net-(D0-Pad2) -> col0
- SW1 pad 1: col1 -> Net-(D1-Pad2)
- SW1 pad 2: Net-(D1-Pad2) -> col1
- SW10 pad 1: col10 -> Net-(D10-Pad2)
- SW10 pad 2: Net-(D10-Pad2) -> col10
- SW11 pad 1: col11 -> Net-(D11-Pad2)
- SW11 pad 2: Net-(D11-Pad2) -> col11
- SW12 pad 1: col12 -> Net-(D12-Pad2)
- SW12 pad 2: Net-(D12-Pad2) -> col12
- SW13 pad 1: col13 -> Net-(D13-Pad2)
- SW13 pad 2: Net-(D13-Pad2) -> col13
- SW14 pad 1: col14 -> Net-(D14-Pad2)
- SW14 pad 2: Net-(D14-Pad2) -> col14
- SW15 pad 1: col0 -> Net-(D15-Pad2)
- SW15 pad 2: Net-(D15-Pad2) -> col0
- SW16 pad 1: col1 -> Net-(D16-Pad2)
- SW16 pad 2: Net-(D16-Pad2) -> col1
- SW17 pad 1: col2 -> Net-(D17-Pad2)
- SW17 pad 2: Net-(D17-Pad2) -> col2
- SW18 pad 1: col3 -> Net-(D18-Pad2)
- SW18 pad 2: Net-(D18-Pad2) -> col3
- SW19 pad 1: col4 -> Net-(D19-Pad2)
- SW19 pad 2: Net-(D19-Pad2) -> col4
- SW2 pad 1: col2 -> Net-(D2-Pad2)
- SW2 pad 2: Net-(D2-Pad2) -> col2
- SW20 pad 1: col5 -> Net-(D20-Pad2)
- SW20 pad 2: Net-(D20-Pad2) -> col5
- SW21 pad 1: col6 -> Net-(D21-Pad2)
- SW21 pad 2: Net-(D21-Pad2) -> col6
- SW22 pad 1: col7 -> Net-(D22-Pad2)
- SW22 pad 2: Net-(D22-Pad2) -> col7
- SW23 pad 1: col8 -> Net-(D23-Pad2)
- SW23 pad 2: Net-(D23-Pad2) -> col8
- SW24 pad 1: col9 -> Net-(D24-Pad2)
- SW24 pad 2: Net-(D24-Pad2) -> col9
- SW25 pad 1: col10 -> Net-(D25-Pad2)
- SW25 pad 2: Net-(D25-Pad2) -> col10
- SW26 pad 1: col11 -> Net-(D26-Pad2)
- SW26 pad 2: Net-(D26-Pad2) -> col11
- SW27 pad 1: col12 -> Net-(D27-Pad2)
- SW27 pad 2: Net-(D27-Pad2) -> col12
- SW28 pad 1: col13 -> Net-(D28-Pad2)
- SW28 pad 2: Net-(D28-Pad2) -> col13
- SW28-2 pad 1: col13 -> Net-(D28-Pad2)
- SW28-2 pad 2: Net-(D28-Pad2) -> col13
- SW29 pad 1: col14 -> Net-(D29-Pad2)
- SW29 pad 2: Net-(D29-Pad2) -> col14
- SW3 pad 1: col3 -> Net-(D3-Pad2)
- SW3 pad 2: Net-(D3-Pad2) -> col3
- SW30 pad 1: col0 -> Net-(D30-Pad2)
- SW30 pad 2: Net-(D30-Pad2) -> col0
- SW31 pad 1: col1 -> Net-(D31-Pad2)
- SW31 pad 2: Net-(D31-Pad2) -> col1
- SW32 pad 1: col2 -> Net-(D32-Pad2)
- SW32 pad 2: Net-(D32-Pad2) -> col2
- SW33 pad 1: col3 -> Net-(D33-Pad2)
- SW33 pad 2: Net-(D33-Pad2) -> col3
- SW34 pad 1: col4 -> Net-(D34-Pad2)
- SW34 pad 2: Net-(D34-Pad2) -> col4
- SW35 pad 1: col5 -> Net-(D35-Pad2)
- SW35 pad 2: Net-(D35-Pad2) -> col5
- SW36 pad 1: col6 -> Net-(D36-Pad2)
- SW36 pad 2: Net-(D36-Pad2) -> col6
- SW37 pad 1: col7 -> Net-(D37-Pad2)
- SW37 pad 2: Net-(D37-Pad2) -> col7
- SW38 pad 1: col8 -> Net-(D38-Pad2)
- SW38 pad 2: Net-(D38-Pad2) -> col8
- SW39 pad 1: col9 -> Net-(D39-Pad2)
- SW39 pad 2: Net-(D39-Pad2) -> col9
- SW4 pad 1: col4 -> Net-(D4-Pad2)
- SW4 pad 2: Net-(D4-Pad2) -> col4
- SW40 pad 1: col10 -> Net-(D40-Pad2)
- SW40 pad 2: Net-(D40-Pad2) -> col10
- SW41 pad 1: col11 -> Net-(D41-Pad2)
- SW41 pad 2: Net-(D41-Pad2) -> col11
- SW42 pad 1: col13 -> Net-(D42-Pad2)
- SW42 pad 2: Net-(D42-Pad2) -> col13
- SW42-2 pad 1: col13 -> Net-(D42-Pad2)
- SW42-2 pad 2: Net-(D42-Pad2) -> col13
- SW43 pad 1: col14 -> Net-(D43-Pad2)
- SW43 pad 2: Net-(D43-Pad2) -> col14
- SW44 pad 1: col0 -> Net-(D44-Pad2)
- SW44 pad 2: Net-(D44-Pad2) -> col0
- SW44-2 pad 1: col0 -> Net-(D44-Pad2)
- SW44-2 pad 2: Net-(D44-Pad2) -> col0
- SW45 pad 1: col1 -> Net-(D45-Pad2)
- SW45 pad 2: Net-(D45-Pad2) -> col1
- SW46 pad 1: col2 -> Net-(D46-Pad2)
- SW46 pad 2: Net-(D46-Pad2) -> col2
- SW47 pad 1: col3 -> Net-(D47-Pad2)
- SW47 pad 2: Net-(D47-Pad2) -> col3
- SW48 pad 1: col4 -> Net-(D48-Pad2)
- SW48 pad 2: Net-(D48-Pad2) -> col4
- SW49 pad 1: col5 -> Net-(D49-Pad2)
- SW49 pad 2: Net-(D49-Pad2) -> col5
- SW5 pad 1: col5 -> Net-(D5-Pad2)
- SW5 pad 2: Net-(D5-Pad2) -> col5
- SW50 pad 1: col6 -> Net-(D50-Pad2)
- SW50 pad 2: Net-(D50-Pad2) -> col6
- SW51 pad 1: col7 -> Net-(D51-Pad2)
- SW51 pad 2: Net-(D51-Pad2) -> col7
- SW52 pad 1: col8 -> Net-(D52-Pad2)
- SW52 pad 2: Net-(D52-Pad2) -> col8
- SW53 pad 1: col9 -> Net-(D53-Pad2)
- SW53 pad 2: Net-(D53-Pad2) -> col9
- SW54 pad 1: col10 -> Net-(D54-Pad2)
- SW54 pad 2: Net-(D54-Pad2) -> col10
- SW55 pad 1: col11 -> Net-(D55-Pad2)
- SW55 pad 2: Net-(D55-Pad2) -> col11
- SW56 pad 1: col12 -> Net-(D56-Pad2)
- SW56 pad 2: Net-(D56-Pad2) -> col12
- SW57 pad 1: col13 -> Net-(D57-Pad2)
- SW57 pad 2: Net-(D57-Pad2) -> col13
- SW58 pad 1: col14 -> Net-(D58-Pad2)
- SW58 pad 2: Net-(D58-Pad2) -> col14
- SW59 pad 1: col0 -> Net-(D59-Pad2)
- SW59 pad 2: Net-(D59-Pad2) -> col0
- SW59-2 pad 1: col0 -> Net-(D59-Pad2)
- SW59-2 pad 2: Net-(D59-Pad2) -> col0
- SW6 pad 1: col6 -> Net-(D6-Pad2)
- SW6 pad 2: Net-(D6-Pad2) -> col6
- SW60 pad 1: col1 -> Net-(D60-Pad2)
- SW60 pad 2: Net-(D60-Pad2) -> col1
- SW60-2 pad 1: col1 -> Net-(D60-Pad2)
- SW60-2 pad 2: Net-(D60-Pad2) -> col1
- SW61 pad 1: col2 -> Net-(D61-Pad2)
- SW61 pad 2: Net-(D61-Pad2) -> col2
- SW62-2 pad 1: col3 -> Net-(D62-Pad2)
- SW62-2 pad 2: Net-(D62-Pad2) -> col3
- SW63 pad 1: col6 -> Net-(D63-Pad2)
- SW63 pad 2: Net-(D63-Pad2) -> col6
- SW63-2 pad 1: col6 -> Net-(D63-Pad2)
- SW63-2 pad 2: Net-(D63-Pad2) -> col6
- SW64 pad 1: col9 -> Net-(D64-Pad2)
- SW64 pad 2: Net-(D64-Pad2) -> col9
- SW64-2 pad 1: col9 -> Net-(D64-Pad2)
- SW64-2 pad 2: Net-(D64-Pad2) -> col9
- SW65 pad 1: col10 -> Net-(D65-Pad2)
- SW65 pad 2: Net-(D65-Pad2) -> col10
- SW65-2 pad 1: col10 -> Net-(D65-Pad2)
- SW65-2 pad 2: Net-(D65-Pad2) -> col10
- SW66 pad 1: col11 -> Net-(D66-Pad2)
- SW66 pad 2: Net-(D66-Pad2) -> col11
- SW67 pad 1: col12 -> Net-(D67-Pad2)
- SW67 pad 2: Net-(D67-Pad2) -> col12
- SW68 pad 1: col13 -> Net-(D68-Pad2)
- SW68 pad 2: Net-(D68-Pad2) -> col13
- SW69 pad 1: col14 -> Net-(D69-Pad2)
- SW69 pad 2: Net-(D69-Pad2) -> col14
- SW7 pad 1: col7 -> Net-(D7-Pad2)
- SW7 pad 2: Net-(D7-Pad2) -> col7
- SW8 pad 1: col8 -> Net-(D8-Pad2)
- SW8 pad 2: Net-(D8-Pad2) -> col8
- SW9 pad 1: col9 -> Net-(D9-Pad2)
- SW9 pad 2: Net-(D9-Pad2) -> col9

Commit message: Adding Stabs back in.
Parts:
- removed ST72: 7U, cftkb:MX-7U-Stabilizer
- added ST13: Stabilizer_Cherry_MX_2u, stabs:Stabilizer_Cherry_MX_2u, F.Cu at (331.4, 106.2)
- added ST42: Stabilizer_Cherry_MX_2u, stabs:Stabilizer_Cherry_MX_2u, F.Cu at (329.1, 144.3)
- added ST59: Stabilizer_Cherry_MX_2u, stabs:Stabilizer_Cherry_MX_2u, F.Cu at (86.2, 163.3)
- added ST63-2: 7U, stabs:Stabilizer_Cherry_MX_7u, F.Cu at (188.7, 182.4)
- ST63: renamed from REF**; footprint cftkb:MX-6.25U-Stabilizer -> stabs:Stabilizer_Cherry_MX_6.25u
- turned ST63 to 180 degrees
